Commit message: Works with one turtlebot

File: ros_ws/src/cwru_turtlebot/urdf/kinect.urdf.xacro (robot description, xacro)
@@ -1,6 +1,6 @@
 <?xml version="1.0"?>
 <robot name="sensor_kinect" xmlns:xacro="http://ros.org/wiki/xacro">
-  <xacro:include filename="$(find turtlebot_description)/urdf/turtlebot_gazebo.urdf.xacro"/>
-  <xacro:include filename="$(find turtlebot_description)/urdf/turtlebot_properties.urdf.xacro"/>
+  <xacro:include filename="$(find cwru_turtlebot)/urdf/turtlebot_gazebo.urdf.xacro"/>
+  <xacro:include filename="$(find cwru_turtlebot)/urdf/turtlebot_properties.urdf.xacro"/>
   <xacro:property name="kinect_cam_py" value="-0.0125"/>
   <!-- Parameterised in part by the values in turtlebot_properties.urdf.xacro -->
@@ -60,5 +60,5 @@
 	<link name="${model_name}/camera_depth_optical_frame"/>
 	<!-- Kinect sensor for simulation -->
-	<turtlebot_sim_3dsensor/>
+	<turtlebot_sim_3dsensor model_name="${model_name}"/>
   </xacro:macro>
 </robot>

File: ros_ws/src/cwru_turtlebot/urdf/turtlebot_gazebo.urdf.xacro (robot description, xacro)
@@ -2,6 +2,6 @@
 <robot name="turtlebot_gazebo" xmlns:xacro="http://ros.org/wiki/xacro">
   <!-- Microsoft Kinect / ASUS Xtion PRO Live for simulation -->
-  <xacro:macro name="turtlebot_sim_3dsensor">
-    <gazebo reference="$(arg model_name)/camera_link">
+  <xacro:macro name="turtlebot_sim_3dsensor" params="model_name">
+    <gazebo reference="${model_name}/camera_link">
       <sensor type="depth" name="camera">
         <always_on>true</always_on>

Commit message: Lots of updates

File: ros_ws/src/cwru_turtlebot/urdf/kinect.urdf.xacro (robot description, xacro)
@@ -5,5 +5,5 @@
   <xacro:property name="kinect_cam_py" value="-0.0125"/>
   <!-- Parameterised in part by the values in turtlebot_properties.urdf.xacro -->
-  <xacro:macro name="sensor_kinect" params="parent model_name">
+  <xacro:macro name="sensor_kinect" params="parent model_name noisy">
     <joint name="${model_name}/camera_rgb_joint" type="fixed">
       <origin xyz="${cam_px} ${kinect_cam_py} ${cam_pz}" rpy="${cam_or} ${cam_op} ${cam_oy}"/>
@@ -60,5 +60,5 @@
 	<link name="${model_name}/camera_depth_optical_frame"/>
 	<!-- Kinect sensor for simulation -->
-	<turtlebot_sim_3dsensor model_name="${model_name}"/>
+	<turtlebot_sim_3dsensor model_name="${model_name}" noisy="${noisy}"/>
   </xacro:macro>
 </robot>

File: ros_ws/src/cwru_turtlebot/urdf/kobuki_hexagons_kinect.urdf.xacro (robot description, xacro)
@@ -9,4 +9,4 @@
   <kobuki model_name="$(arg model_name)"/>
   <stack_hexagons parent="$(arg model_name)/base_link" model_name="$(arg model_name)"/>
-  <sensor_kinect  parent="$(arg model_name)/base_link" model_name="$(arg model_name)"/>
+  <sensor_kinect  parent="$(arg model_name)/base_link" model_name="$(arg model_name)" noisy="$(arg noisy)"/>
 </robot>

File: ros_ws/src/cwru_turtlebot/urdf/turtlebot_gazebo.urdf.xacro (robot description, xacro)
@@ -2,5 +2,5 @@
 <robot name="turtlebot_gazebo" xmlns:xacro="http://ros.org/wiki/xacro">
     <!-- Microsoft Kinect / ASUS Xtion PRO Live for simulation -->
-    <xacro:macro name="turtlebot_sim_3dsensor" params="model_name">
+    <xacro:macro name="turtlebot_sim_3dsensor" params="model_name noisy">
         <gazebo reference="${model_name}/camera_link">
             <sensor type="depth" name="camera">
@@ -18,10 +18,12 @@
                         <far>8.0</far>
                     </clip>
-                    <noise>
-                        <!-- Noise parameters taken from Gazebo documentation recommendation -->
-                        <type>gaussian</type>
-                        <mean>0.0</mean>
-                        <stddev>0.007</stddev>
-                    </noise>
+                    <xacro:if value="${noisy}">
+                        <noise>
+                            <!-- Noise parameters taken from Gazebo documentation recommendation -->
+                            <type>gaussian</type>
+                            <mean>0.0</mean>
+                            <stddev>0.007</stddev>
+                        </noise>
+                    </xacro:if>
                 </camera>
                 <plugin name="kinect_camera_controller" filename="libgazebo_ros_openni_kinect.so">
