Commit message: Adds control of IMU noise via noisy parameter

File: ros_ws/src/cwru_turtlebot/urdf/kobuki.urdf.xacro (robot description, xacro)
@@ -10,5 +10,5 @@
   <xacro:include filename="$(find cwru_turtlebot)/urdf/kobuki_gazebo.urdf.xacro"/>
   <!-- Kobuki -->
-  <xacro:macro name="kobuki" params="model_name">
+  <xacro:macro name="kobuki" params="model_name noisy">
     <link name="${model_name}/base_footprint"/>
     <!--
@@ -209,5 +209,5 @@
     </link>
     <!-- Kobuki Gazebo simulation details -->
-    <kobuki_sim model_name="${model_name}"/>
+    <kobuki_sim model_name="${model_name}" noisy="${noisy}"/>
   </xacro:macro>
 </robot>

File: ros_ws/src/cwru_turtlebot/urdf/kobuki_gazebo.urdf.xacro (robot description, xacro)
@@ -1,5 +1,5 @@
 <?xml version="1.0"?>
 <robot name="kobuki_sim" xmlns:xacro="http://ros.org/wiki/xacro">
-    <xacro:macro name="kobuki_sim" params="model_name">
+    <xacro:macro name="kobuki_sim" params="model_name noisy">
         <gazebo reference="${model_name}/wheel_left_link">
             <mu1>1.0</mu1>
@@ -142,19 +142,21 @@
                 <visualize>false</visualize>
                 <imu>
-                    <noise>
-                        <type>gaussian</type>
-                        <rate>
-                            <mean>0.0</mean>
-                            <stddev>${0.0014*0.0014}</stddev> <!-- 0.25 x 0.25 (deg/s) -->
-                            <bias_mean>0.0</bias_mean>
-                            <bias_stddev>0.0</bias_stddev>
-                        </rate>
-                        <accel> <!-- not used in the plugin and real robot, hence using tutorial values -->
-                            <mean>0.0</mean>
-                            <stddev>1.7e-2</stddev>
-                            <bias_mean>0.1</bias_mean>
-                            <bias_stddev>0.001</bias_stddev>
-                        </accel>
-                    </noise>
+                    <xacro:if value="${noisy}">
+                        <noise>
+                            <type>gaussian</type>
+                            <rate>
+                                <mean>0.0</mean>
+                                <stddev>${0.0014*0.0014}</stddev> <!-- 0.25 x 0.25 (deg/s) -->
+                                <bias_mean>0.0</bias_mean>
+                                <bias_stddev>0.0</bias_stddev>
+                            </rate>
+                            <accel> <!-- not used in the plugin and real robot, hence using tutorial values -->
+                                <mean>0.0</mean>
+                                <stddev>1.7e-2</stddev>
+                                <bias_mean>0.1</bias_mean>
+                                <bias_stddev>0.001</bias_stddev>
+                            </accel>
+                        </noise>
+                    </xacro:if>
                 </imu>
             </sensor>

File: ros_ws/src/cwru_turtlebot/urdf/kobuki_hexagons_kinect.urdf.xacro (robot description, xacro)
@@ -7,5 +7,5 @@
 <robot name="turtlebot" xmlns:xacro="http://ros.org/wiki/xacro">
   <xacro:include filename="$(find cwru_turtlebot)/urdf/turtlebot_library.urdf.xacro"/>
-  <kobuki model_name="$(arg model_name)"/>
+  <kobuki model_name="$(arg model_name)" noisy="$(arg noisy)"/>
   <stack_hexagons parent="$(arg model_name)/base_link" model_name="$(arg model_name)"/>
   <sensor_kinect  parent="$(arg model_name)/base_link" model_name="$(arg model_name)" noisy="$(arg noisy)"/>
